File: toy_car_atmega8_board.kicad_pcb (KiCad board)
At the start: 2 copper layers, 50 x 50 mm, 16 parts, among them J1 Conn_01x06_Pin, J2 Conn_01x08_Pin, J3 Conn_01x06_Pin, J4 Conn_01x06_Pin, J5 Conn_01x02_Pin, SW1 SW_Push, U1 ATmega8A-P, Y1 16Mhz

Commit message: Added further changes
Parts:
- moved J3 5.21 mm to (117.5, 77.3)
- moved J4 5.18 mm to (117.5, 55.8)
- moved R1 4.57 mm to (110.5, 38.9)
- moved C5 2.55 mm to (119.2, 60.8), turned to 180 degrees
Routing:
- net /MOSI: track 58.8 -> 48.5 mm
- net /MISO: track 65.9 -> 57.4 mm
- net /SCK: track 74.3 -> 67.3 mm
- net GND: track 188.3 -> 181.8 mm
- net /C1_ADC1: track 10.4 -> 4.82 mm
- net /C0_ADC0: track 10.4 -> 4.82 mm
- net /C2_ADC2: track 10.4 -> 4.82 mm
- net /SDA: track 10.4 -> 4.82 mm
- net /C3_ADC3: track 10.4 -> 4.82 mm
- net /SCL: track 10.4 -> 4.82 mm
- net /B2_SS_OC1B: track 10.5 -> 5.35 mm
- net /B0_ICP1: track 18.8 -> 13.7 mm
- net /B1_OC1A: track 10.5 -> 5.35 mm
- net Net-(D1-K): track 27.4 -> 23.5 mm
- net /D5_T1: track 33.8 -> 31.9 mm
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Other:
- board size 50 x 50 mm -> 46 x 50 mm

Commit message: Updated pcb
Parts:
- moved C2 1.02 mm to (91.0, 68.5)
- moved SW1 0.97 mm to (97.9, 49.2)
- moved C3 0.51 mm to (81.9, 73.7)
- moved C4 0.38 mm to (87.2, 47.2)
Connections:
- J1 pad 1: /VCC -> /RESET
- J1 pad 2: /RESET -> /VCC
Routing:
- net GND: track 181.8 -> 278.1 mm, vias 0 -> 3
- net /RESET: track 58.4 -> 68.4 mm, vias 0 -> 2
- net /VCC: track 116.8 -> 115.1 mm
- net /D6_AIN0: track 30.3 -> 29.6 mm
- net /RXD: track 29.1 -> 28.4 mm
- net Net-(U1-PB7/XTAL2): track 13.2 -> 12.6 mm
Other:
- board text added: "+"
- board text added: "GND"
